File: KiCad/GR_Twin_T_Filter.kicad_pcb (KiCad board)
At the start: 2 copper layers, 46.9 x 41.4 mm, 35 parts, among them J1 Conn_01x03, J2 Conn_01x02, J3 Conn_01x02, J4 Conn_01x02, J5 Conn_01x03, U1 LM358

Commit message: Add files via upload
Connections:
- J1 pad 1: GNDREF -> /Ext.Use
- J1 pad 2: Net-(J1-Pad2) -> /Ext.Use
- J1 pad 3: Net-(C2-Pad1) -> GNDREF
- R3 pad 2: Net-(J1-Pad2) -> /Ext.Use
- R5 pad 2: GNDREF -> /Ext.Use
- R5 pad 3: GNDREF -> /Ext.Use
Routing:
- net /Ext.Use: track 0.00 -> 48.2 mm, vias 0 -> 1
- net Net-(J1-Pad2): track 15.8 -> 0.00 mm, vias 1 -> 0
- net Net-(C2-Pad1): track 21.9 -> 10.5 mm
Other:
- board text added: "Ext."
- board text removed: "Tee"
